File: Eagle files/SoundLab.brd (EAGLE design)
At the start: 157.5 x 96.5 mm, 138 parts, among them IC1 LM555D, IC2 LM3900D, IC3 LM3900D, IC4 LM324D, IC5 LM555D, IC6 LM386M-1, J7 5.5x2.1mm Barrel, P1 200k, P10 200k, P11 200k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

Commit message: R100->R55
Parts:
- renumbered R100 to R55
Changed lines of the file:
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@@
 <attribute name="VALUE" x="22.352" y="69.85" size="1.27" layer="28" rot="MR270"/>
 </element>
-<element name="R100" library="microbuilder" package="_0805MP" value="100k" x="22.225" y="75.8825" smashed="yes" rot="MR270">
+<element name="R55" library="microbuilder" package="_0805MP" value="100k" x="22.225" y="75.8825" smashed="yes" rot="MR270">
 <attribute name="NAME" x="23.8125" y="77.47" size="0.8128" layer="26" ratio="18" rot="MR270"/>
 <attribute name="VALUE" x="23.495" y="77.47" size="0.4064" layer="28" ratio="10" rot="MR270"/>
@@
 </signal>
 <signal name="N$1">
-<contactref element="R100" pad="2"/>
+<contactref element="R55" pad="2"/>
 <contactref element="R17" pad="2"/>
 <contactref element="IC3" pad="1"/>
@@
 <signal name="N$14">
 <contactref element="P2" pad="P$2"/>
-<contactref element="R100" pad="1"/>
+<contactref element="R55" pad="1"/>
 <wire x1="22.225" y1="76.8985" x2="22.225" y2="80.3275" width="0.4064" layer="16"/>
 <wire x1="74.93" y1="90.17" x2="76.2" y2="88.9" width="0.4064" layer="16"/>
